Commit message: Sync

File: rbx_vol_1/rbx1_dynamixels/urdf/head.xacro (robot description, xacro)
@@ -1,5 +1,5 @@
 <?xml version="1.0"?>
 <robot>
-  <include filename="$(find rbx_dynamixels)/urdf/head_hardware.xacro" />
+  <include filename="$(find rbx1_dynamixels)/urdf/head_hardware.xacro" />
   <macro name="turtlebot_head" params="parent color *origin">
     <link name="head_base_link" />
@@ -48,5 +48,5 @@
         <origin xyz="0 0 0 " rpy="0 0 0" />
         <geometry>
-          <mesh filename="package://rbx_dynamixels/meshes/kinect.dae" />
+          <mesh filename="package://rbx1_dynamixels/meshes/kinect.dae" />
         </geometry>
       </visual>

File: rbx_vol_1/rbx1_dynamixels/urdf/head_hardware.xacro (robot description, xacro)
@@ -27,5 +27,5 @@
         <origin xyz=" 0 0 0 " rpy="0 0 0" />
         <geometry>
-          <mesh filename="package://rbx_dynamixels/meshes/F10.${MESH_EXT}" scale="${M_SCALE} ${M_SCALE} ${M_SCALE}"/>
+          <mesh filename="package://rbx1_dynamixels/meshes/F10.${MESH_EXT}" scale="${M_SCALE} ${M_SCALE} ${M_SCALE}"/>
         </geometry>
         <material name="${color}"/>
@@ -56,5 +56,5 @@
         <origin xyz=" 0 0 0 " rpy="0 0 0" />
         <geometry>
-          <mesh filename="package://rbx_dynamixels/meshes/F3.${MESH_EXT}" scale="${M_SCALE} ${M_SCALE} ${M_SCALE}"/>
+          <mesh filename="package://rbx1_dynamixels/meshes/F3.${MESH_EXT}" scale="${M_SCALE} ${M_SCALE} ${M_SCALE}"/>
         </geometry>
         <material name="${color}"/>
@@ -85,5 +85,5 @@
         <origin xyz=" 0 0 0 " rpy="0 0 0" />
         <geometry>
-          <mesh filename="package://rbx_dynamixels/meshes/ax12_box.${MESH_EXT}" scale="${M_SCALE} ${M_SCALE} ${M_SCALE}"/>
+          <mesh filename="package://rbx1_dynamixels/meshes/ax12_box.${MESH_EXT}" scale="${M_SCALE} ${M_SCALE} ${M_SCALE}"/>
         </geometry>
         <material name="black"/>
@@ -116,5 +116,5 @@
         <origin xyz=" 0 0 0 " rpy="0 0 0" />
         <geometry>
-          <mesh filename="package://rbx_dynamixels/meshes/F3.${MESH_EXT}" scale="${M_SCALE} ${M_SCALE} ${M_SCALE}"/>
+          <mesh filename="package://rbx1_dynamixels/meshes/F3.${MESH_EXT}" scale="${M_SCALE} ${M_SCALE} ${M_SCALE}"/>
         </geometry>
         <material name="${color}"/>
@@ -147,5 +147,5 @@
         <origin xyz=" 0 0 0 " rpy="0 0 0" />
         <geometry>
-          <mesh filename="package://rbx_dynamixels/meshes/F4.${MESH_EXT}" scale="${M_SCALE} ${M_SCALE} ${M_SCALE}"/>
+          <mesh filename="package://rbx1_dynamixels/meshes/F4.${MESH_EXT}" scale="${M_SCALE} ${M_SCALE} ${M_SCALE}"/>
         </geometry>
         <material name="${color}"/>

File: rbx_vol_1/rbx1_dynamixels/urdf/pi_turtlebot.xacro (robot description, xacro)
@@ -5,6 +5,6 @@
     xmlns:interface="http://playerstage.sourceforge.net/gazebo/xmlschema/#interface">
     <!-- Included URDF Files -->
-    <include filename="$(find rbx_dynamixels)/urdf/turtlebot.xacro" />
-    <include filename="$(find rbx_dynamixels)/urdf/head.xacro" />
+    <include filename="$(find rbx1_dynamixels)/urdf/turtlebot.xacro" />
+    <include filename="$(find rbx1_dynamixels)/urdf/head.xacro" />
     <turtlebot />
     <turtlebot_head parent="plate_3_link" color="white">

File: rbx_vol_1/rbx1_dynamixels/urdf/turtlebot.xacro (robot description, xacro)
@@ -1,5 +1,5 @@
 <?xml version="1.0"?>
 <robot>
-  <include filename="$(find rbx_dynamixels)/urdf/turtlebot_hardware.xacro" />
+  <include filename="$(find rbx1_dynamixels)/urdf/turtlebot_hardware.xacro" />
   <include filename="$(find turtlebot_description)/urdf/gazebo.urdf.xacro"/>
   <property name="M_PI" value="3.14159"/>
@@ -388,5 +388,5 @@
       <origin xyz=" 0 0 0 " rpy="0 0 0" />
       <geometry>
-        <mesh filename="package://rbx_dynamixels/meshes/kinect.dae"/>
+        <mesh filename="package://rbx1_dynamixels/meshes/kinect.dae"/>
       </geometry>
     </visual>

File: rbx_vol_1/rbx1_dynamixels/urdf/turtlebot_hardware.xacro (robot description, xacro)
@@ -20,5 +20,5 @@
         <origin xyz=" 0 0 0 " rpy="0 0 0" />
         <geometry>
-          <mesh filename="package://pi_tb_description/meshes/68-02403-125_Spacer.dae" scale="${M_SCALE} ${M_SCALE} ${M_SCALE}" />
+          <mesh filename="package://rbx1_dynamixels/meshes/68-02403-125_Spacer.dae" scale="${M_SCALE} ${M_SCALE} ${M_SCALE}" />
         </geometry>
       </visual>
@@ -48,5 +48,5 @@
         <origin xyz=" 0 0 0 " rpy="0 0 0" />
         <geometry>
-          <mesh filename="package://pi_tb_description/meshes/68-04552-1000-RA_Turtlebot_M-F_Standoff.dae" scale="${M_SCALE} ${M_SCALE} ${M_SCALE}"/>
+          <mesh filename="package://rbx1_dynamixels/meshes/68-04552-1000-RA_Turtlebot_M-F_Standoff.dae" scale="${M_SCALE} ${M_SCALE} ${M_SCALE}"/>
         </geometry>
       </visual>
@@ -76,5 +76,5 @@
         <origin xyz=" 0 0 0 " rpy="0 0 0" />
         <geometry>
-          <mesh filename="package://pi_tb_description/meshes/68-04552-2000-RA_Turtlebot_M-F_Standoff.dae" scale="${M_SCALE} ${M_SCALE} ${M_SCALE}"/>
+          <mesh filename="package://rbx1_dynamixels/meshes/68-04552-2000-RA_Turtlebot_M-F_Standoff.dae" scale="${M_SCALE} ${M_SCALE} ${M_SCALE}"/>
         </geometry>
       </visual>
@@ -104,5 +104,5 @@
         <origin xyz=" 0 0 0 " rpy="0 0 0" />
         <geometry>
-          <mesh filename="package://pi_tb_description/meshes/68-04552-2000-RA_Turtlebot_M-F_Standoff.dae" scale="${M_SCALE} ${M_SCALE} ${M_SCALE*1.5}"/>
+          <mesh filename="package://rbx1_dynamixels/meshes/68-04552-2000-RA_Turtlebot_M-F_Standoff.dae" scale="${M_SCALE} ${M_SCALE} ${M_SCALE*1.5}"/>
         </geometry>
       </visual>
@@ -132,5 +132,5 @@
         <origin xyz=" 0 0 0 " rpy="0 0 0" />
         <geometry>
-          <mesh filename="package://pi_tb_description/meshes/68-02421-8000-RA_Turtlebot_F-F_Standoff.dae" scale="${M_SCALE} ${M_SCALE} ${M_SCALE}"/>
+          <mesh filename="package://rbx1_dynamixels/meshes/68-02421-8000-RA_Turtlebot_F-F_Standoff.dae" scale="${M_SCALE} ${M_SCALE} ${M_SCALE}"/>
         </geometry>
       </visual>
