Commit message: Removed reference to pi_tb_description in rbx1_description/turtlebot.xacro

File: rbx_vol_1/rbx1_description/urdf/turtlebot.xacro (robot description, xacro)
@@ -1,5 +1,5 @@
 <?xml version="1.0"?>
 <robot>
-  <include filename="$(find pi_tb_description)/urdf/turtlebot_hardware.xacro" />
+  <include filename="$(find rbx1_description)/urdf/turtlebot_hardware.xacro" />
   <include filename="$(find turtlebot_description)/urdf/gazebo.urdf.xacro"/>
   <material name="Green">
@@ -379,5 +379,5 @@
       <origin xyz=" 0 0 0 " rpy="0 0 0" />
       <geometry>
-        <mesh filename="package://pi_tb_description/meshes/kinect.dae"/>
+        <mesh filename="package://rbx1_description/meshes/kinect.dae"/>
       </geometry>
     </visual>
